File: vic2020mainboard/vic2020cpu.sch (KiCad schematic (older format))
At the start: 40 parts, among them J1 A15 KERNAL/BASIC SELECT, J2 A14 Kernel/Basic Select, SW1 RAM ENABLE, U1 7402, U10 74LS133, U11 74LS02, U12 AS6C1008-55PCN, U13 27512, U2 74LS138, U24 74ALS32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

Commit message: Correct SVIDEO connector footprint
Parts:
- C2: symbol Device:CTRIM -> Vic2020mainboard-rescue:CTRIM-Device
- FB1, FB2, FB3: symbol Device:Ferrite_Bead_Small -> Vic2020mainboard-rescue:Ferrite_Bead_Small-Device
- U3: symbol Timer:LM555 -> Vic2020mainboard-rescue:LM555-Timer
Changed lines of the file:
@@
 $EndComp
 $Comp
-L Timer:LM555 U?
+L Vic2020mainboard-rescue:LM555-Timer U?
 U 1 1 5F669AD1
 P 1850 4300
@@
 	1250 900  800  900
 $Comp
-L Device:CTRIM C2
+L Vic2020mainboard-rescue:CTRIM-Device C2
 U 1 1 5F669BC8
 P 1900 900
@@
 $EndComp
 $Comp
-L Device:Ferrite_Bead_Small FB3
+L Vic2020mainboard-rescue:Ferrite_Bead_Small-Device FB3
 U 1 1 5F9EA778
 P 8000 5100
@@
 	8450 5100 9050 5100
 $Comp
-L Device:Ferrite_Bead_Small FB2
+L Vic2020mainboard-rescue:Ferrite_Bead_Small-Device FB2
 U 1 1 5FA26CDB
 P 7000 6150
@@
 	6700 6150 6900 6150
 $Comp
-L Device:Ferrite_Bead_Small FB1
+L Vic2020mainboard-rescue:Ferrite_Bead_Small-Device FB1
 U 1 1 5FA803BA
 P 5950 6150

Commit message: update PCB
Parts:
- C4: footprint Capacitor_THT:C_Rect_L7.0mm_W2.0mm_P5.00mm -> Capacitor_THT:CP_Radial_D4.0mm_P2.00mm
- U12: symbol as6c1008-55pcn:AS6C1008-55PCN -> Vic2020mainboard-rescue:AS6C1008-55PCN-as6c1008-55pcn
Changed lines of the file:
@@
 F 0 "C4" H 2615 4896 50  0000 L CNN
 F 1 "10uf" H 2615 4805 50  0000 L CNN
-F 2 "Capacitor_THT:C_Rect_L7.0mm_W2.0mm_P5.00mm" H 2538 4700 50  0001 C CNN
+F 2 "Capacitor_THT:CP_Radial_D4.0mm_P2.00mm" H 2538 4700 50  0001 C CNN
 F 3 "~" H 2500 4850 50  0001 C CNN
 	1    2500 4850
@@
 	7650 650  7750 650
 $Comp
-L as6c1008-55pcn:AS6C1008-55PCN U12
+L Vic2020mainboard-rescue:AS6C1008-55PCN-as6c1008-55pcn U12
 U 1 1 6016B148
 P 7650 1750
