File: vic2020mainboard/VIC2020DISPLAY.sch (KiCad schematic (older format))
At the start: 46 parts, among them J3 FONT SELECT, J4 Chroma Disconnect, J5 SVIDEO Out, J6 Audio Out, J7 Video Out, Q1 2sc1959, Q2 2SC1815, U14 74LS245, U15 74LS245, U16 74LS245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

Commit message: Correct SVIDEO connector footprint
Parts:
- C11, C37, C38, C39, C9: symbol Device:CP -> Vic2020mainboard-rescue:CP-Device
- FB4, FB5, FB6, FB7, FB8, FB9: symbol Device:Ferrite_Bead_Small -> Vic2020mainboard-rescue:Ferrite_Bead_Small-Device
- RV1: symbol Device:R_POT -> Vic2020mainboard-rescue:R_POT-Device
Changed lines of the file:
@@
 $EndComp
 $Comp
-L Device:CP C11
+L Vic2020mainboard-rescue:CP-Device C11
 U 1 1 608440DF
 P 10500 1350
+AR Path="/608440DF" Ref="C11"  Part="1"
+AR Path="/5F5BC33E/608440DF" Ref="C11"  Part="1"
 F 0 "C11" V 10245 1350 50  0000 C CNN
 F 1 "1uf" V 10336 1350 50  0000 C CNN
@@
 $EndComp
 $Comp
-L Device:R_POT RV1
+L Vic2020mainboard-rescue:R_POT-Device RV1
 U 1 1 6085CD64
 P 8900 2800
@@
 L power:GND #PWR0167
 U 1 1 60F8D94E
-P 7550 4900
-F 0 "#PWR0167" H 7550 4650 50  0001 C CNN
-F 1 "GND" H 7555 4727 50  0000 C CNN
-F 2 "" H 7550 4900 50  0001 C CNN
-F 3 "" H 7550 4900 50  0001 C CNN
-	1    7550 4900
+P 7950 5400
+F 0 "#PWR0167" H 7950 5150 50  0001 C CNN
+F 1 "GND" H 7955 5227 50  0000 C CNN
+F 2 "" H 7950 5400 50  0001 C CNN
+F 3 "" H 7950 5400 50  0001 C CNN
+	1    7950 5400
 	1    0    0    -1
 $EndComp
@@
 NoConn ~ 5200 2350
 $Comp
-L Device:Ferrite_Bead_Small FB7
+L Vic2020mainboard-rescue:Ferrite_Bead_Small-Device FB7
 U 1 1 5F767278
 P 6300 850
@@
 $EndComp
 $Comp
-L Device:Ferrite_Bead_Small FB8
+L Vic2020mainboard-rescue:Ferrite_Bead_Small-Device FB8
 U 1 1 5F768674
 P 6300 1000
@@
 	5400 850  5500 850
 $Comp
-L Device:CP C9
+L Vic2020mainboard-rescue:CP-Device C9
 U 1 1 5F792C3C
 P 6850 750
+AR Path="/5F792C3C" Ref="C9"  Part="1"
+AR Path="/5F5BC33E/5F792C3C" Ref="C9"  Part="1"
 F 0 "C9" H 7000 650 50  0000 R CNN
 F 1 "2.2uF" H 6800 650 50  0000 R CNN
@@
 $EndComp
 $Comp
-L Device:CP C37
+L Vic2020mainboard-rescue:CP-Device C37
 U 1 1 5F794472
 P 7250 750
+AR Path="/5F794472" Ref="C37"  Part="1"
+AR Path="/5F5BC33E/5F794472" Ref="C37"  Part="1"
 F 0 "C37" H 7350 850 50  0000 R CNN
 F 1 ".47uF" H 7200 650 50  0000 R CNN
@@
 Connection ~ 8100 1000
 $Comp
-L Device:CP C38
+L Vic2020mainboard-rescue:CP-Device C38
 U 1 1 5F96202A
 P 8950 2150
+AR Path="/5F96202A" Ref="C38"  Part="1"
+AR Path="/5F5BC33E/5F96202A" Ref="C38"  Part="1"
 F 0 "C38" H 8850 2450 50  0000 L CNN
 F 1 "10uF" H 8850 2350 50  0000 L CNN
@@
 	8950 2000 9300 2000
 $Comp
-L Device:CP C39
+L Vic2020mainboard-rescue:CP-Device C39
 U 1 1 5F96349E
 P 9450 2750
+AR Path="/5F96349E" Ref="C39"  Part="1"
+AR Path="/5F5BC33E/5F96349E" Ref="C39"  Part="1"
 F 0 "C39" V 9300 2750 50  0000 C CNN
 F 1 "47uF" V 9600 2700 50  0000 C CNN
@@
 $EndComp
 $Comp
-L Device:Ferrite_Bead_Small FB9
+L Vic2020mainboard-rescue:Ferrite_Bead_Small-Device FB9
 U 1 1 5F9637C5
 P 7750 3000
@@
 	7500 3000 7600 3000
 $Comp
-L Device:Ferrite_Bead_Small FB6
+L Vic2020mainboard-rescue:Ferrite_Bead_Small-Device FB6
 U 1 1 5F9795E0
 P 4950 2200
@@
 	4850 2200 4650 2200
 $Comp
-L Device:Ferrite_Bead_Small FB5
+L Vic2020mainboard-rescue:Ferrite_Bead_Small-Device FB5
 U 1 1 5F98DF3B
 P 4950 1300
@@
 $EndComp
 $Comp
-L Device:Ferrite_Bead_Small FB4
+L Vic2020mainboard-rescue:Ferrite_Bead_Small-Device FB4
 U 1 1 5F98E82C
 P 4800 1400
@@
 Text GLabel 9100 3650 2    50   Input ~ 0
 SVIDC
-Text GLabel 8100 5250 2    50   Input ~ 0
+Text GLabel 8100 4400 2    50   Input ~ 0
 VIDEOOUT
-Text GLabel 8100 4400 2    50   Input ~ 0
+Text GLabel 7550 4750 0    50   Input ~ 0
 SVIDC
 Wire Wire Line
@@
 Wire Wire Line
 	8100 5250 8100 5150
-Wire Wire Line
-	7800 4750 7550 4750
-Wire Wire Line
-	7550 4750 7550 4800
-Wire Wire Line
-	7800 4950 7800 4800
-Wire Wire Line
-	7800 4800 7550 4800
-Connection ~ 7550 4800
-Wire Wire Line
-	7550 4800 7550 4900
 Wire Wire Line
 	9050 2800 9100 2800
@@
 Wire Wire Line
 	8250 3650 8150 3650
+Wire Wire Line
+	7950 5250 7950 5400
+Wire Wire Line
+	8100 5250 7950 5250
+Wire Wire Line
+	7800 5250 7800 4950
+Connection ~ 7950 5250
+Wire Wire Line
+	7950 5250 7800 5250
+Wire Wire Line
+	7800 4750 7550 4750
 $EndSCHEMATC

Commit message: update PCB
Parts:
- C40: footprint Capacitor_THT:CP_Radial_D4.0mm_P2.00mm -> Capacitor_THT:C_Rect_L7.0mm_W2.0mm_P5.00mm
- U17: symbol as6c1008-55pcn:AS6C1008-55PCN -> Vic2020mainboard-rescue:AS6C1008-55PCN-as6c1008-55pcn
- U20: symbol 6560:6560 -> Vic2020mainboard-rescue:6560-6560
Changed lines of the file:
@@
 $EndComp
 $Comp
-L 6560:6560 U20
+L Vic2020mainboard-rescue:6560-6560 U20
 U 1 1 6083B46F
 P 5800 2500
+AR Path="/6083B46F" Ref="U20"  Part="1"
+AR Path="/5F5BC33E/6083B46F" Ref="U20"  Part="1"
 F 0 "U20" H 5800 2700 50  0000 C CNN
 F 1 "6560" H 5850 2550 50  0000 C CIB
@@
 	4000 2900 4150 2900
 $Comp
-L as6c1008-55pcn:AS6C1008-55PCN U17
+L Vic2020mainboard-rescue:AS6C1008-55PCN-as6c1008-55pcn U17
 U 1 1 607D5355
 P 3500 3800
@@
 F 0 "C40" V 7748 3650 50  0000 C CNN
 F 1 ".1uf" V 7839 3650 50  0000 C CNN
-F 2 "Capacitor_THT:CP_Radial_D4.0mm_P2.00mm" H 8038 3500 50  0001 C CNN
+F 2 "Capacitor_THT:C_Rect_L7.0mm_W2.0mm_P5.00mm" H 8038 3500 50  0001 C CNN
 F 3 "~" H 8000 3650 50  0001 C CNN
 	1    8000 3650

Commit message: Fix SVIDEO (again)
Connections:
- net SVIDC: now also J5.4; no longer J5.3
- net VIDEOOUT: now also J5.3; no longer J5.4
Changed lines of the file:
@@
 Text GLabel 9100 3650 2    50   Input ~ 0
 SVIDC
-Text GLabel 8100 4400 2    50   Input ~ 0
+Text GLabel 7550 4750 0    50   Input ~ 0
 VIDEOOUT
-Text GLabel 7550 4750 0    50   Input ~ 0
+Text GLabel 8100 4400 0    50   Input ~ 0
 SVIDC
 Wire Wire Line
