File: vic2020mainboard/Vic2020mainboard.kicad_pcb (KiCad board)
At the start: 2 copper layers, 357.8 x 124.5 mm, 144 parts, among them J1 A15 KERNAL/BASIC SELECT, J10 5v Regulated, J11 Conn_02x08_Odd_Even, J12 Conn_02x22_Row_Letter_First, J13 IEC, J14 Joystick 1, J2 A14 KERNAL/BASIC SELECT, J3 FONT SELECT, J4 Chroma Disconnect, J5 SVIDEO, J6 Audio Out, J7 Video Out, J8 Keyboard, J9 LED, Q1 2sc1959, Q2 2SC1815, SW1 RAM ENABLE, SW3 Expansion Port, U1 7402, U10 74LS133, U11 74LS02, U12 AS6C1008-55PCN, U13 27512, U14 74LS245, U15 74LS245, U16 74LS245, U17 AS6C1008-55PCN, U18 74LS245, U19 2764, U2 74LS138, U20 6560, U21 W65C22NxP, U22 W65C22NxP, U23 74LS245, U24 74ALS32, U3 LM555, U4 7406, U5 74LS133, U6 74LS138, U7 W65C02SxP, U8 74LS00, U9 74LS04, Y1 Crystal

Commit message: Correct SVIDEO connector footprint
Parts:
- J13: value IEC -> IEC Port
- J2: value A14 KERNAL/BASIC SELECT -> A14 Kernel/Basic Select
- J5: value SVIDEO -> SVIDEO Out
- moved G*** 226.3 mm to (64.7, 203.2)
- moved G*** 0.83 mm to (279.1, 166.3)
Connections:
- J5 pad 1: VIDEOOUT -> GND
- J5 pad 3: GND -> SVIDC
- J5 pad 4: SVIDC -> VIDEOOUT
Routing:
- net VIDEOOUT: track 97.7 -> 105.8 mm
- net SVIDC: track 30.5 -> 35.4 mm
- net GND: track 1414.9 -> 1415.5 mm
Other:
- board text added: "DAN WERNER VIC-2020 4/3/2020 - V 1.1"
- board text removed: "DAN WERNER VIC-2020 12/5/2020 - V 1.0"
Changed lines of the file:
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@@
     (thickness 1.6)
     (drawings 24)
-    (tracks 6322)
+    (tracks 6330)
     (zones 0)
     (modules 144)
@@
   (page USLedger)
   (layers
-    (0 F.Cu signal)
-    (31 B.Cu signal)
+    (0 F.Cu signal hide)
+    (31 B.Cu signal hide)
     (32 B.Adhes user)
     (33 F.Adhes user)
@@
     (add_net "Net-(FB9-Pad1)")
     (add_net "Net-(J1-Pad2)")
+    (add_net "Net-(J12-Pada14)")
+    (add_net "Net-(J12-Pada15)")
+    (add_net "Net-(J12-Pada16)")
+    (add_net "Net-(J12-Pada20)")
+    (add_net "Net-(J12-Padb21)")
     (add_net "Net-(J13-Pad3)")
     (add_net "Net-(J2-Pad2)")
     (add_net "Net-(J3-Pad2)")
+    (add_net "Net-(J8-Pad2)")
     (add_net "Net-(J9-Pad2)")
     (add_net "Net-(R11-Pad1)")
@@
     (add_net "Net-(U11-Pad4)")
     (add_net "Net-(U11-Pad6)")
+    (add_net "Net-(U12-Pad1)")
+    (add_net "Net-(U16-Pad11)")
+    (add_net "Net-(U16-Pad9)")
+    (add_net "Net-(U17-Pad1)")
     (add_net "Net-(U18-Pad19)")
+    (add_net "Net-(U19-Pad26)")
+    (add_net "Net-(U20-Pad1)")
+    (add_net "Net-(U20-Pad36)")
+    (add_net "Net-(U23-Pad11)")
+    (add_net "Net-(U23-Pad12)")
+    (add_net "Net-(U23-Pad13)")
+    (add_net "Net-(U23-Pad14)")
+    (add_net "Net-(U23-Pad15)")
+    (add_net "Net-(U23-Pad5)")
+    (add_net "Net-(U23-Pad6)")
+    (add_net "Net-(U23-Pad7)")
+    (add_net "Net-(U23-Pad8)")
+    (add_net "Net-(U23-Pad9)")
     (add_net "Net-(U24-Pad8)")
     (add_net "Net-(U3-Pad3)")
+    (add_net "Net-(U3-Pad5)")
+    (add_net "Net-(U6-Pad12)")
+    (add_net "Net-(U6-Pad13)")
+    (add_net "Net-(U6-Pad14)")
+    (add_net "Net-(U6-Pad15)")
+    (add_net "Net-(U7-Pad35)")
     (add_net "Net-(U8-Pad3)")
     (add_net O1)
@@
   )
   (module logo:we_vsmall_neg (layer F.Cu)
-    (at 291 204.8)
+    (at 64.74 203.22)
     (fp_text reference G*** (at 0 0) (layer F.SilkS) hide
       (effects (font (size 1.524 1.524) (thickness 0.3)))
@@
   )
   (module logo:viclogo (layer F.Cu)
-    (at 279.9 166.3)
+    (at 279.07 166.28)
     (fp_text reference G*** (at 0 0) (layer F.SilkS) hide
       (effects (font (size 1.524 1.524) (thickness 0.3)))
@@
       (effects (font (size 1.001764 1.001764) (thickness 0.135)))
     )
-    (fp_text value IEC (at -12.2 6.3 270) (layer F.SilkS)
+    (fp_text value "IEC Port" (at -12.2 6.3 270) (layer F.SilkS)
       (effects (font (size 3 3) (thickness 0.015)))
     )
@@
       (effects (font (size 0.800449 0.800449) (thickness 0.015)))
     )
-    (fp_text value SVIDEO (at 10.9 -0.4 90) (layer F.SilkS)
+    (fp_text value "SVIDEO Out" (at 10.9 -0.4 90) (layer F.SilkS)
       (effects (font (size 3 3) (thickness 0.1415)))
     )
@@
     (fp_circle (center -3.4 4.8) (end -3.3 4.8) (layer F.SilkS) (width 0.2))
     (pad 1 thru_hole rect (at -3.35 0) (size 1.398 1.398) (drill 0.89) (layers *.Cu *.Mask)
-      (net 16 VIDEOOUT))
-    (pad 3 thru_hole circle (at -3.35 2.49) (size 1.398 1.398) (drill 0.89) (layers *.Cu *.Mask)
       (net 1 GND))
+    (pad 3 thru_hole circle (at -3.35 2.49) (size 1.398 1.398) (drill 0.89) (layers *.Cu *.Mask)
+      (net 177 SVIDC))
     (pad 2 thru_hole circle (at 3.35 0) (size 1.398 1.398) (drill 0.89) (layers *.Cu *.Mask)
       (net 1 GND))
     (pad 4 thru_hole circle (at 3.35 2.49) (size 1.398 1.398) (drill 0.89) (layers *.Cu *.Mask)
-      (net 177 SVIDC))
+      (net 16 VIDEOOUT))
     (pad 5 thru_hole circle (at 0 -3.81) (size 3.306 3.306) (drill 2.29) (layers *.Cu *.Mask))
     (pad 6 thru_hole circle (at 6.76 -3) (size 3.306 3.306) (drill 2.29) (layers *.Cu *.Mask))
@@
       (effects (font (size 1 1) (thickness 0.15)))
     )
-    (fp_text value "A14 KERNAL/BASIC SELECT" (at -2.8 1.8 180) (layer F.SilkS)
+    (fp_text value "A14 Kernel/Basic Select" (at -2.8 1.8 180) (layer F.SilkS)
       (effects (font (size 1 1) (thickness 0.15)))
     )
@@
     (effects (font (size 1.6 1) (thickness 0.15)))
   )
-  (gr_text "DAN WERNER\nVIC-2020\n12/5/2020 - V 1.0" (at 213.7 204.4) (layer F.SilkS)
+  (gr_text "DAN WERNER\nVIC-2020 \n4/3/2020 - V 1.1" (at 213.7 204.4) (layer F.SilkS)
     (effects (font (size 2 2) (thickness 0.15)))
   )
@@
   (segment (start 242.3998 169.2807) (end 242.3997 169.2807) (width 1) (layer B.Cu) (net 1))
   (segment (start 242.3997 169.2807) (end 242.3997 182.62) (width 1) (layer B.Cu) (net 1))
-  (segment (start 118.85 97.59) (end 115.6485 97.59) (width 1) (layer B.Cu) (net 1))
   (segment (start 115.6485 97.59) (end 107.7061 105.5324) (width 1) (layer B.Cu) (net 1))
   (segment (start 107.7061 105.5324) (end 110.4 108.2263) (width 1) (layer B.Cu) (net 1))
@@
   (segment (start 99.3282 102.5251) (end 104.6988 102.5251) (width 1) (layer B.Cu) (net 1))
   (segment (start 104.6988 102.5251) (end 107.7061 105.5324) (width 1) (layer B.Cu) (net 1))
-  (segment (start 125.55 95.1) (end 123.06 97.59) (width 1) (layer B.Cu) (net 1))
-  (segment (start 123.06 97.59) (end 118.85 97.59) (width 1) (layer B.Cu) (net 1))
   (segment (start 99.3282 102.5251) (end 99.3282 102.2689) (width 1) (layer B.Cu) (net 1))
   (segment (start 99.3282 102.2689) (end 95.5813 98.522) (width 1) (layer B.Cu) (net 1))
@@
   (segment (start 196.975 90.1497) (end 191.7006 90.1497) (width 1) (layer B.Cu) (net 1))
   (segment (start 191.7006 90.1497) (end 191.0503 90.8) (width 1) (layer B.Cu) (net 1))
-  (segment (start 146.8 101.5) (end 131.95 101.5) (width 1) (layer B.Cu) (net 1))
-  (segment (start 131.95 101.5) (end 125.55 95.1) (width 1) (layer B.Cu) (net 1))
   (segment (start 372.3 175.7) (end 372.3 177.5) (width 1) (layer B.Cu) (net 1))
   (segment (start 372.3 177.5) (end 358 191.8) (width 1) (layer B.Cu) (net 1))
@@
   (segment (start 77.72 151.3) (end 77.72 149.7497) (width 1) (layer B.Cu) (net 1))
   (via (at 237.2545 159.2429) (size 0.8) (layers F.Cu B.Cu) (net 1))
+  (segment (start 146.8 101.5) (end 131.95 101.5) (width 1) (layer B.Cu) (net 1))
+  (segment (start 131.95 101.5) (end 125.55 95.1) (width 1) (layer B.Cu) (net 1))
+  (segment (start 115.6485 97.59) (end 115.6485 97.4615) (width 0.25) (layer B.Cu) (net 1))
+  (segment (start 115.6485 97.4615) (end 117.03 96.08) (width 0.25) (layer B.Cu) (net 1))
+  (segment (start 118.85 96.049) (end 118.85 95.1) (width 0.25) (layer B.Cu) (net 1))
+  (segment (start 118.819 96.08) (end 118.85 96.049) (width 0.25) (layer B.Cu) (net 1))
+  (segment (start 117.03 96.08) (end 118.819 96.08) (width 0.25) (layer B.Cu) (net 1))
+  (segment (start 118.85 95.1) (end 125.55 95.1) (width 0.25) (layer B.Cu) (net 1))
   (segment (start 301.2607 159.9941) (end 300.6503 160.6045) (width 0.25) (layer F.Cu) (net 2))
   (segment (start 300.6503 160.6045) (end 285.9059 160.6045) (width 0.25) (layer F.Cu) (net 2))
@@
   (segment (start 88.32 113.4) (end 89.4453 113.4) (width 0.25) (layer F.Cu) (net 15))
   (segment (start 131.2 119.78) (end 130.0747 119.78) (width 0.25) (layer F.Cu) (net 15))
-  (segment (start 97.1 96.4) (end 98.2003 96.4) (width 0.25) (layer B.Cu) (net 16))
-  (segment (start 118.85 95.1) (end 99.5003 95.1) (width 0.25) (layer B.Cu) (net 16))
-  (segment (start 99.5003 95.1) (end 98.2003 96.4) (width 0.25) (layer B.Cu) (net 16))
   (segment (start 53.2 113.8353) (end 53.0656 113.8353) (width 0.25) (layer B.Cu) (net 16))
   (segment (start 53.0656 113.8353) (end 51.4877 115.4132) (width 0.25) (layer B.Cu) (net 16))
@@
   (segment (start 97.1 96.4) (end 95.9997 96.4) (width 0.25) (layer F.Cu) (net 16))
   (via (at 55.4274 103.4011) (size 0.8) (layers F.Cu B.Cu) (net 16))
+  (segment (start 97.1 96.4) (end 111.29 96.4) (width 0.25) (layer F.Cu) (net 16))
+  (segment (start 111.29 96.4) (end 114.29 99.4) (width 0.25) (layer F.Cu) (net 16))
+  (segment (start 123.74 99.4) (end 125.55 97.59) (width 0.25) (layer F.Cu) (net 16))
+  (segment (start 114.29 99.4) (end 123.74 99.4) (width 0.25) (layer F.Cu) (net 16))
   (segment (start 253.0787 94.234) (end 253.0787 93.8574) (width 0.25) (layer B.Cu) (net 17))
   (segment (start 253.0787 93.8574) (end 251.3749 92.1536) (width 0.25) (layer B.Cu) (net 17))
@@
   (via (at 242.6863 167.4381) (size 0.8) (layers F.Cu B.Cu) (net 176))
   (segment (start 115.4 123.9) (end 125.55 113.75) (width 0.25) (layer B.Cu) (net 177))
-  (segment (start 125.55 113.75) (end 125.55 97.59) (width 0.25) (layer B.Cu) (net 177))
+  (segment (start 119.548999 98.288999) (end 123.128999 98.288999) (width 0.25) (layer B.Cu) (net 177))
+  (segment (start 118.85 97.59) (end 119.548999 98.288999) (width 0.25) (layer B.Cu) (net 177))
+  (segment (start 123.128999 98.288999) (end 125.57 100.73) (width 0.25) (layer B.Cu) (net 177))
+  (segment (start 125.57 113.73) (end 125.55 113.75) (width 0.25) (layer B.Cu) (net 177))
+  (segment (start 125.57 100.73) (end 125.57 113.73) (width 0.25) (layer B.Cu) (net 177))
   (segment (start 237.1257 167.2526) (end 241.5406 167.2526) (width 0.25) (layer F.Cu) (net 178))
   (segment (start 241.5406 167.2526) (end 242.0805 166.7127) (width 0.25) (layer F.Cu) (net 178))
@@
     (polygon
       (pts
-        (xy 390.9 208.9) (xy 36.9 208.3) (xy 37.8 88.1) (xy 391.7 87.6)
+        (xy 390.8 209.02) (xy 37.22 208.25) (xy 37.71 87.99) (xy 37.73 87.99) (xy 391.42 87.81)
       )
     )

Commit message: update PCB
Parts:
- removed G***: LOGO, logo:we_vsmall_neg
- removed G***: LOGO, logo:viclogo
- C4: footprint Capacitor_THT:C_Rect_L7.0mm_W2.0mm_P5.00mm -> Capacitor_THT:CP_Radial_D4.0mm_P2.00mm
- C40: footprint Capacitor_THT:CP_Radial_D4.0mm_P2.00mm -> Capacitor_THT:C_Rect_L7.0mm_W2.0mm_P5.00mm
- J13: value IEC Port -> IEC
- J5: value SVIDEO Out -> SVIDEO
- moved C4 4.33 mm to (360.6, 108.9), turned to 270 degrees
- moved C40 3.33 mm to (108.6, 128.0)
Routing:
- net Net-(C40-Pad1): track 19.5 -> 16.2 mm
- net A1: track 402.8 -> 403.5 mm
- net Net-(C4-Pad1): vias 0 -> 1
- net GND: vias 1 -> 2
Other:
- board text added: "FOR HOBBYEST/EXPERIMENTAL USE ONLY"
- board text added: "https://bitbucket.org/danwerner21/vic2020/"

Commit message: Fix SVIDEO (again)
Parts:
- J13: value IEC -> IEC Port
- J5: value SVIDEO -> SVIDEO Out
Connections:
- J5 pad 3: SVIDC -> VIDEOOUT
- J5 pad 4: VIDEOOUT -> SVIDC
Routing:
- net VIDEOOUT: track 105.8 -> 99.1 mm
- net SVIDC: track 35.4 -> 30.5 mm
Other:
- board text added: "DAN WERNER VIC-2020 8/15/2021 - V 1.2"
- board text removed: "DAN WERNER VIC-2020 4/3/2020 - V 1.1"
Changed lines of the file:
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@@
     (thickness 1.6)
     (drawings 26)
-    (tracks 6345)
+    (tracks 6344)
     (zones 0)
     (modules 142)
@@
   (page USLedger)
   (layers
-    (0 F.Cu signal hide)
-    (31 B.Cu signal hide)
+    (0 F.Cu signal)
+    (31 B.Cu signal)
     (32 B.Adhes user)
-    (33 F.Adhes user)
+    (33 F.Adhes user hide)
     (34 B.Paste user)
     (35 F.Paste user)
@@
       (effects (font (size 1.001764 1.001764) (thickness 0.135)))
     )
-    (fp_text value IEC (at -12.2 6.3 270) (layer F.SilkS)
+    (fp_text value "IEC Port" (at -12.2 6.3 270) (layer F.SilkS)
       (effects (font (size 3 3) (thickness 0.3)))
     )
@@
       (effects (font (size 0.800449 0.800449) (thickness 0.015)))
     )
-    (fp_text value SVIDEO (at 10.9 -0.4 90) (layer F.SilkS)
+    (fp_text value "SVIDEO Out" (at 10.9 -0.4 90) (layer F.SilkS)
       (effects (font (size 3 3) (thickness 0.3)))
     )
@@
       (net 1 GND))
     (pad 3 thru_hole circle (at -3.35 2.49) (size 1.398 1.398) (drill 0.89) (layers *.Cu *.Mask)
-      (net 177 SVIDC))
+      (net 16 VIDEOOUT))
     (pad 2 thru_hole circle (at 3.35 0) (size 1.398 1.398) (drill 0.89) (layers *.Cu *.Mask)
       (net 1 GND))
     (pad 4 thru_hole circle (at 3.35 2.49) (size 1.398 1.398) (drill 0.89) (layers *.Cu *.Mask)
-      (net 16 VIDEOOUT))
+      (net 177 SVIDC))
     (pad 5 thru_hole circle (at 0 -3.81) (size 3.306 3.306) (drill 2.29) (layers *.Cu *.Mask))
     (pad 6 thru_hole circle (at 6.76 -3) (size 3.306 3.306) (drill 2.29) (layers *.Cu *.Mask))
@@
     (effects (font (size 1.6 1) (thickness 0.15)))
   )
-  (gr_text "DAN WERNER\nVIC-2020 \n4/3/2020 - V 1.1" (at 213.7 204.4) (layer F.SilkS)
+  (gr_text "DAN WERNER\nVIC-2020 \n8/15/2021 - V 1.2" (at 213.7 204.4) (layer F.SilkS)
     (effects (font (size 2 2) (thickness 0.15)))
   )
@@
   (segment (start 97.1 96.4) (end 111.29 96.4) (width 0.25) (layer F.Cu) (net 16))
   (segment (start 111.29 96.4) (end 114.29 99.4) (width 0.25) (layer F.Cu) (net 16))
-  (segment (start 123.74 99.4) (end 125.55 97.59) (width 0.25) (layer F.Cu) (net 16))
-  (segment (start 114.29 99.4) (end 123.74 99.4) (width 0.25) (layer F.Cu) (net 16))
+  (segment (start 117.04 99.4) (end 118.85 97.59) (width 0.25) (layer F.Cu) (net 16))
+  (segment (start 114.29 99.4) (end 117.04 99.4) (width 0.25) (layer F.Cu) (net 16))
   (segment (start 253.0787 94.234) (end 253.0787 93.8574) (width 0.25) (layer B.Cu) (net 17))
   (segment (start 253.0787 93.8574) (end 251.3749 92.1536) (width 0.25) (layer B.Cu) (net 17))
@@
   (segment (start 231.52 179.34) (end 231.52 180.4653) (width 0.25) (layer B.Cu) (net 176))
   (via (at 242.6863 167.4381) (size 0.8) (layers F.Cu B.Cu) (net 176))
-  (segment (start 115.4 123.9) (end 125.55 113.75) (width 0.25) (layer B.Cu) (net 177))
-  (segment (start 119.548999 98.288999) (end 123.128999 98.288999) (width 0.25) (layer B.Cu) (net 177))
-  (segment (start 118.85 97.59) (end 119.548999 98.288999) (width 0.25) (layer B.Cu) (net 177))
-  (segment (start 123.128999 98.288999) (end 125.57 100.73) (width 0.25) (layer B.Cu) (net 177))
+  (segment (start 125.55 113.75) (end 115.4 123.9) (width 0.25) (layer B.Cu) (net 177))
   (segment (start 125.57 113.73) (end 125.55 113.75) (width 0.25) (layer B.Cu) (net 177))
   (segment (start 125.57 100.73) (end 125.57 113.73) (width 0.25) (layer B.Cu) (net 177))
+  (segment (start 125.55 97.59) (end 125.55 100.71) (width 0.25) (layer B.Cu) (net 177))
+  (segment (start 125.55 100.71) (end 125.57 100.73) (width 0.25) (layer B.Cu) (net 177))
   (segment (start 237.1257 167.2526) (end 241.5406 167.2526) (width 0.25) (layer F.Cu) (net 178))
   (segment (start 241.5406 167.2526) (end 242.0805 166.7127) (width 0.25) (layer F.Cu) (net 178))
