File: vic2020keyboard/vic2020keyboard.kicad_pcb (KiCad board)
At the start: 2 copper layers, 341.2 x 124.5 mm, 78 parts, among them J1 Conn_01x20_Male, SW1 0, SW10 9, SW11 PLUS, SW12 MINUS, SW13 POUND, SW14 AT, SW15 ASTERISK, SW16 COLON, SW17 SEMICOLON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

Commit message: updates
Parts:
- removed G***: LOGO, logo:we_small_neg
- removed G***: LOGO, logo:viclogo
